File: asd/_saved_PCBdisplay.sch (KiCad schematic (older format))
At the start: 25 parts, among them J1 CONN_02X20, SW1 SW_DIP_x02, SW2 SW_DIP_x02, U1 MC34064D

Commit message: commit
Parts:
- added D?: LED, symbol LED
- added R?: R, symbol R
- added U?: MC34064D, symbol MC34064D
Connections:
- wire segments 71 -> 78
Other:
- moved on the sheet: BZ1, D8, R8, R9, SW1
Changed lines of the file:
@@
 L R R8
 U 1 1 5953AD82
-P 1300 4600
-F 0 "R8" V 1380 4600 50  0000 C CNN
-F 1 "R" V 1300 4600 50  0000 C CNN
-F 2 "" V 1230 4600 50  0001 C CNN
-F 3 "" H 1300 4600 50  0001 C CNN
-	1    1300 4600
+P 1300 4650
+F 0 "R8" V 1380 4650 50  0000 C CNN
+F 1 "R" V 1300 4650 50  0000 C CNN
+F 2 "" V 1230 4650 50  0001 C CNN
+F 3 "" H 1300 4650 50  0001 C CNN
+	1    1300 4650
 	-1   0    0    1
 $EndComp
@@
 L GND #PWR1
 U 1 1 5953B40E
-P 1300 4400
-F 0 "#PWR1" H 1300 4150 50  0001 C CNN
-F 1 "GND" H 1300 4250 50  0000 C CNN
-F 2 "" H 1300 4400 50  0001 C CNN
-F 3 "" H 1300 4400 50  0001 C CNN
-	1    1300 4400
+P 1300 4450
+F 0 "#PWR1" H 1300 4200 50  0001 C CNN
+F 1 "GND" H 1300 4300 50  0000 C CNN
+F 2 "" H 1300 4450 50  0001 C CNN
+F 3 "" H 1300 4450 50  0001 C CNN
+	1    1300 4450
 	-1   0    0    1
 $EndComp
@@
 	5250 2250 5250 2100
 Wire Wire Line
-	1300 4450 1300 4400
+	1300 4500 1300 4450
 $Comp
 L LED D6
@@
 L LED D8
 U 1 1 5953B956
-P 1300 4900
-F 0 "D8" H 1300 5000 50  0000 C CNN
-F 1 "LED" H 1300 4800 50  0000 C CNN
-F 2 "" H 1300 4900 50  0001 C CNN
-F 3 "" H 1300 4900 50  0001 C CNN
-	1    1300 4900
+P 1300 4950
+F 0 "D8" H 1300 5050 50  0000 C CNN
+F 1 "LED" H 1300 4850 50  0000 C CNN
+F 2 "" H 1300 4950 50  0001 C CNN
+F 3 "" H 1300 4950 50  0001 C CNN
+	1    1300 4950
 	0    1    1    0
 $EndComp
@@
 	5250 3100 5250 2850
 Wire Wire Line
-	1300 5100 1300 5050
+	1300 5150 1300 5100
 $Comp
 L GND #PWR11
@@
 L SW_DIP_x02 SW1
 U 1 1 59562F17
-P 2350 4950
-F 0 "SW1" H 2350 5200 50  0000 C CNN
-F 1 "SW_DIP_x02" H 2350 4800 50  0000 C CNN
-F 2 "" H 2350 4950 50  0001 C CNN
-F 3 "" H 2350 4950 50  0001 C CNN
-	1    2350 4950
+P 2350 5000
+F 0 "SW1" H 2350 5250 50  0000 C CNN
+F 1 "SW_DIP_x02" H 2350 4850 50  0000 C CNN
+F 2 "" H 2350 5000 50  0001 C CNN
+F 3 "" H 2350 5000 50  0001 C CNN
+	1    2350 5000
 	0    1    1    0
 $EndComp
@@
 Text Notes 3350 4200 0    118  ~ 0
 Header Raspberry Pi 3
-NoConn ~ 2350 5250
-NoConn ~ 2350 4650
-Wire Wire Line
-	2450 4500 2450 4650
-Wire Wire Line
-	2450 5250 2450 5300
+NoConn ~ 2350 5300
+NoConn ~ 2350 4700
+Wire Wire Line
+	2450 4550 2450 4650
+Wire Wire Line
+	2450 4650 2450 4700
+Wire Wire Line
+	2450 5300 2450 5350
 $Comp
 L R R9
 U 1 1 59566B6C
-P 2700 4600
-F 0 "R9" V 2780 4600 50  0000 C CNN
-F 1 "R" V 2700 4600 50  0000 C CNN
-F 2 "" V 2630 4600 50  0001 C CNN
-F 3 "" H 2700 4600 50  0001 C CNN
-	1    2700 4600
-	0    1    1    0
-$EndComp
-Wire Wire Line
-	2450 4600 2550 4600
-Wire Wire Line
-	2850 4600 2900 4600
+P 2700 4650
+F 0 "R9" V 2780 4650 50  0000 C CNN
+F 1 "R" V 2700 4650 50  0000 C CNN
+F 2 "" V 2630 4650 50  0001 C CNN
+F 3 "" H 2700 4650 50  0001 C CNN
+	1    2700 4650
+	0    1    1    0
+$EndComp
+Wire Wire Line
+	2450 4650 2550 4650
+Wire Wire Line
+	2850 4650 2900 4650
 $Comp
 L GND #PWR4
 U 1 1 59566EAD
-P 2450 5300
-F 0 "#PWR4" H 2450 5050 50  0001 C CNN
-F 1 "GND" H 2450 5150 50  0000 C CNN
-F 2 "" H 2450 5300 50  0001 C CNN
-F 3 "" H 2450 5300 50  0001 C CNN
-	1    2450 5300
+P 2450 5350
+F 0 "#PWR4" H 2450 5100 50  0001 C CNN
+F 1 "GND" H 2450 5200 50  0000 C CNN
+F 2 "" H 2450 5350 50  0001 C CNN
+F 3 "" H 2450 5350 50  0001 C CNN
+	1    2450 5350
 	0    -1   -1   0
 $EndComp
@@
 L GND #PWR7
 U 1 1 59566F01
-P 2900 4600
-F 0 "#PWR7" H 2900 4350 50  0001 C CNN
-F 1 "GND" H 2900 4450 50  0000 C CNN
-F 2 "" H 2900 4600 50  0001 C CNN
-F 3 "" H 2900 4600 50  0001 C CNN
-	1    2900 4600
+P 2900 4650
+F 0 "#PWR7" H 2900 4400 50  0001 C CNN
+F 1 "GND" H 2900 4500 50  0000 C CNN
+F 2 "" H 2900 4650 50  0001 C CNN
+F 3 "" H 2900 4650 50  0001 C CNN
+	1    2900 4650
 	1    0    0    -1
 $EndComp
@@
 	-1   0    0    1
 $EndComp
-Connection ~ 2450 4600
-Text Label 2450 4500 1    60   ~ 0
+Connection ~ 2450 4650
+Text Label 2450 4550 1    60   ~ 0
 GPIO
 Wire Notes Line
-	3050 3950 3050 5400
+	3050 3950 3050 5550
 Wire Notes Line
 	3000 5400 3000 5400
@@
 	3050 3950 2000 3950
 Wire Notes Line
-	2000 3950 2000 5400
-Wire Notes Line
-	2000 5400 3050 5400
-Wire Notes Line
-	1850 5400 800  5400
-Wire Notes Line
-	800  5400 800  3950
+	2000 3950 2000 5550
+Wire Notes Line
+	2000 5550 3050 5550
+Wire Notes Line
+	1850 5550 800  5550
+Wire Notes Line
+	800  5550 800  3950
 Wire Notes Line
 	800  3950 1850 3950
 Wire Notes Line
-	1850 3950 1850 5400
+	1850 3950 1850 5550
 $Comp
 L MC34064D U1
@@
 Wire Wire Line
 	6550 5700 6550 5800
-Text Label 2100 5300 1    60   ~ 0
-GPIO
-Wire Wire Line
-	2500 6100 2550 6100
+Wire Wire Line
+	2500 6300 2550 6300
 $Comp
 L Buzzer BZ1
 U 1 1 59569201
-P 2650 6000
-F 0 "BZ1" H 2800 6050 50  0000 L CNN
-F 1 "Buzzer" H 2800 5950 50  0000 L BNN
-F 2 "" V 2625 6100 50  0001 C CNN
-F 3 "" V 2625 6100 50  0001 C CNN
-	1    2650 6000
+P 2650 6200
+F 0 "BZ1" H 2800 6250 50  0000 L CNN
+F 1 "Buzzer" H 2800 6150 50  0000 L BNN
+F 2 "" V 2625 6300 50  0001 C CNN
+F 3 "" V 2625 6300 50  0001 C CNN
+	1    2650 6200
 	0    -1   -1   0
 $EndComp
 Wire Wire Line
-	2750 6100 2750 6150
+	2750 6300 2750 6350
 $Comp
 L GND #PWR6
 U 1 1 59569E95
-P 2750 6150
-F 0 "#PWR6" H 2750 5900 50  0001 C CNN
-F 1 "GND" H 2750 6000 50  0000 C CNN
-F 2 "" H 2750 6150 50  0001 C CNN
-F 3 "" H 2750 6150 50  0001 C CNN
-	1    2750 6150
+P 2750 6350
+F 0 "#PWR6" H 2750 6100 50  0001 C CNN
+F 1 "GND" H 2750 6200 50  0000 C CNN
+F 2 "" H 2750 6350 50  0001 C CNN
+F 3 "" H 2750 6350 50  0001 C CNN
+	1    2750 6350
 	1    0    0    -1
 $EndComp
 Wire Notes Line
-	800  5550 3050 5550
-Wire Notes Line
-	3050 5550 3050 6550
+	800  5700 3050 5700
+Wire Notes Line
+	3050 5700 3050 6550
 Wire Notes Line
 	3050 6550 800  6550
 Wire Notes Line
-	800  6550 800  5550
+	800  6550 800  5700
 Wire Wire Line
 	6200 5350 6250 5350
@@
 Text Notes 2050 4100 0    59   ~ 0
 Botó STOP alarma
-Text Notes 850  5700 0    79   ~ 0
+Text Notes 850  5850 0    79   ~ 0
 Brunzidor volum alarma
 $Comp
@@
 NoConn ~ 6300 6950
 Wire Wire Line
-	6400 6800 6400 6950
+	6400 6800 6400 6900
+Wire Wire Line
+	6400 6900 6400 6950
 Wire Wire Line
 	6400 7550 6400 7600
@@
 Brillantor Display\n
 NoConn ~ 6300 7550
+$Comp
+L MC34064D U?
+U 1 1 59567B60
+P 1950 6250
+F 0 "U?" H 2000 6450 50  0000 C CNN
+F 1 "MC34064D" H 2250 6054 50  0000 C CNN
+F 2 "" H 1950 6250 50  0001 C CNN
+F 3 "" H 1950 6250 50  0001 C CNN
+	1    1950 6250
+	-1   0    0    1
+$EndComp
+$Comp
+L GND #PWR?
+U 1 1 59567B66
+P 1950 5950
+F 0 "#PWR?" H 1950 5700 50  0001 C CNN
+F 1 "GND" H 1950 5800 50  0000 C CNN
+F 2 "" H 1950 5950 50  0001 C CNN
+F 3 "" H 1950 5950 50  0001 C CNN
+	1    1950 5950
+	0    -1   -1   0
+$EndComp
+Wire Wire Line
+	1600 6300 1500 6300
+Wire Wire Line
+	1950 5950 1950 6000
+Wire Wire Line
+	2300 6300 2500 6300
+$Comp
+L R R?
+U 1 1 59568BBC
+P 4500 2400
+F 0 "R?" V 4580 2400 50  0000 C CNN
+F 1 "R" V 4500 2400 50  0000 C CNN
+F 2 "" V 4430 2400 50  0001 C CNN
+F 3 "" H 4500 2400 50  0001 C CNN
+	1    4500 2400
+	-1   0    0    1
+$EndComp
+$Comp
+L GND #PWR?
+U 1 1 59568BC2
+P 4500 2100
+F 0 "#PWR?" H 4500 1850 50  0001 C CNN
+F 1 "GND" H 4500 1950 50  0000 C CNN
+F 2 "" H 4500 2100 50  0001 C CNN
+F 3 "" H 4500 2100 50  0001 C CNN
+	1    4500 2100
+	-1   0    0    1
+$EndComp
+Wire Wire Line
+	4500 2250 4500 2100
+$Comp
+L LED D?
+U 1 1 59568BC9
+P 4500 2700
+F 0 "D?" H 4500 2800 50  0000 C CNN
+F 1 "LED" H 4500 2600 50  0000 C CNN
+F 2 "" H 4500 2700 50  0001 C CNN
+F 3 "" H 4500 2700 50  0001 C CNN
+	1    4500 2700
+	0    1    1    0
+$EndComp
+Wire Wire Line
+	4500 3100 4500 2850
 $EndSCHEMATC
