File: PCB display/PCBdisplay.kicad_pcb (KiCad board)
At the start: 2 copper layers, 25 parts, among them J1 CONN_02X20

Commit message: commit
Parts:
- added SW1: SW_DIP_x02, Buttons_Switches_THT:SW_PUSH-12mm, F.Cu at (102.9, 107.3)
- added SW2: SW_DIP_x02, Buttons_Switches_THT:SW_PUSH-12mm, F.Cu at (202.6, 99.1)
- R1, R10, R11, R2, R3, R4, R5, R6, R7, R8, R9: footprint Resistors_SMD:R_0201 -> Resistors_THT:R_Axial_DIN0204_L3.6mm_D1.6mm_P7.62mm_Horizontal
- moved R9 55.0 mm to (98.4, 114.9), turned to 90 degrees
- moved RV2 46.6 mm to (106.0, 88.3), turned to 270 degrees
- moved R10 38.9 mm to (219.7, 106.7), turned to 90 degrees
- moved DS1 35.1 mm to (183.5, 122.6)
- moved RV1 30.5 mm to (210.8, 123.8), turned to 90 degrees
- moved D8 27.3 mm to (88.9, 114.9)
- moved D6 26.1 mm to (184.2, 79.4)
- moved D7 26.1 mm to (179.1, 79.4)
- moved D9 25.5 mm to (173.4, 79.4)
- moved J1 25.3 mm to (142.2, 106.0)
- moved BZ1 24.9 mm to (89.5, 91.4), turned to 180 degrees
- moved D2 24.7 mm to (156.2, 78.7)
- moved D1 24.7 mm to (161.3, 78.7)
- moved D3 24.7 mm to (151.1, 78.7)
- moved R8 24.2 mm to (93.3, 114.9), turned to 90 degrees
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