File: PCB display/PCBdisplay.sch (KiCad schematic (older format))
At the start: 25 parts, among them J1 CONN_02X20, SW1 SW_DIP_x02, SW2 SW_DIP_x02, U1 MC34064D

Commit message: commited
Parts:
- removed U1: MC34064D, symbol MC34064D
- added D9: LED, LEDs:LED_D3.0mm_Horizontal_O1.27mm_Z2.0mm, symbol LED
- added R11: R, Resistors_SMD:R_0201, symbol R
- added RV2: POT, Potentiometers:Potentiometer_Alps_RK09K_Vertical, symbol POT
- BZ1: footprint (none) -> Buzzers_Beepers:BUZZER
- D1, D2, D3, D4, D5, D6, D7, D8: footprint (none) -> LEDs:LED_D3.0mm_Horizontal_O1.27mm_Z2.0mm
- J1: footprint (none) -> Pin_Headers:Pin_Header_Angled_2x20_Pitch2.00mm
- R1, R10, R2, R3, R4, R5, R6, R7, R8, R9: footprint (none) -> Resistors_SMD:R_0201
- RV1: footprint (none) -> Potentiometers:Potentiometer_Alps_RK09K_Vertical
Connections:
- net labels added: CONT_DISP
- net labels removed: +5V, GPIO, GPIO13, GPIO21, GPIO22, GPIO5, GPIO6, GPIO9
- wire segments 71 -> 65
- no-connect marks 23 -> 25
Other:
- moved on the sheet: BZ1, R10, RV1, SW2

Commit message: commit
Parts:
- R1, R10, R11, R2, R3, R4, R5, R6, R7, R8, R9: footprint Resistors_SMD:R_0201 -> Resistors_THT:R_Axial_DIN0204_L3.6mm_D1.6mm_P7.62mm_Horizontal
- SW1, SW2: footprint (none) -> Buttons_Switches_THT:SW_PUSH-12mm
Changed lines of the file:
@@
 LIBS:switches
 LIBS:Power_Management
+LIBS:PCBdisplay-cache
 EELAYER 26 0
 EELAYER END
@@
 F 0 "R1" V 3530 2300 50  0000 C CNN
 F 1 "R" V 3450 2300 50  0000 C CNN
-F 2 "Resistors_SMD:R_0201" V 3380 2300 50  0001 C CNN
+F 2 "Resistors_THT:R_Axial_DIN0204_L3.6mm_D1.6mm_P7.62mm_Horizontal" V 3380 2300 50  0001 C CNN
 F 3 "" H 3450 2300 50  0001 C CNN
 	1    3450 2300
@@
 F 0 "R2" V 3130 2300 50  0000 C CNN
 F 1 "R" V 3050 2300 50  0000 C CNN
-F 2 "Resistors_SMD:R_0201" V 2980 2300 50  0001 C CNN
+F 2 "Resistors_THT:R_Axial_DIN0204_L3.6mm_D1.6mm_P7.62mm_Horizontal" V 2980 2300 50  0001 C CNN
 F 3 "" H 3050 2300 50  0001 C CNN
 	1    3050 2300
@@
 F 0 "R3" V 2680 2300 50  0000 C CNN
 F 1 "R" V 2600 2300 50  0000 C CNN
-F 2 "Resistors_SMD:R_0201" V 2530 2300 50  0001 C CNN
+F 2 "Resistors_THT:R_Axial_DIN0204_L3.6mm_D1.6mm_P7.62mm_Horizontal" V 2530 2300 50  0001 C CNN
 F 3 "" H 2600 2300 50  0001 C CNN
 	1    2600 2300
@@
 F 0 "R4" V 2230 2300 50  0000 C CNN
 F 1 "R" V 2150 2300 50  0000 C CNN
-F 2 "Resistors_SMD:R_0201" V 2080 2300 50  0001 C CNN
+F 2 "Resistors_THT:R_Axial_DIN0204_L3.6mm_D1.6mm_P7.62mm_Horizontal" V 2080 2300 50  0001 C CNN
 F 3 "" H 2150 2300 50  0001 C CNN
 	1    2150 2300
@@
 F 0 "R5" V 1780 2300 50  0000 C CNN
 F 1 "R" V 1700 2300 50  0000 C CNN
-F 2 "Resistors_SMD:R_0201" V 1630 2300 50  0001 C CNN
+F 2 "Resistors_THT:R_Axial_DIN0204_L3.6mm_D1.6mm_P7.62mm_Horizontal" V 1630 2300 50  0001 C CNN
 F 3 "" H 1700 2300 50  0001 C CNN
 	1    1700 2300
@@
 F 0 "R6" V 6130 2400 50  0000 C CNN
 F 1 "R" V 6050 2400 50  0000 C CNN
-F 2 "Resistors_SMD:R_0201" V 5980 2400 50  0001 C CNN
+F 2 "Resistors_THT:R_Axial_DIN0204_L3.6mm_D1.6mm_P7.62mm_Horizontal" V 5980 2400 50  0001 C CNN
 F 3 "" H 6050 2400 50  0001 C CNN
 	1    6050 2400
@@
 F 0 "R7" V 5330 2400 50  0000 C CNN
 F 1 "R" V 5250 2400 50  0000 C CNN
-F 2 "Resistors_SMD:R_0201" V 5180 2400 50  0001 C CNN
+F 2 "Resistors_THT:R_Axial_DIN0204_L3.6mm_D1.6mm_P7.62mm_Horizontal" V 5180 2400 50  0001 C CNN
 F 3 "" H 5250 2400 50  0001 C CNN
 	1    5250 2400
@@
 F 0 "R8" V 1380 4600 50  0000 C CNN
 F 1 "R" V 1300 4600 50  0000 C CNN
-F 2 "Resistors_SMD:R_0201" V 1230 4600 50  0001 C CNN
+F 2 "Resistors_THT:R_Axial_DIN0204_L3.6mm_D1.6mm_P7.62mm_Horizontal" V 1230 4600 50  0001 C CNN
 F 3 "" H 1300 4600 50  0001 C CNN
 	1    1300 4600
@@
 F 0 "SW1" H 2350 5200 50  0000 C CNN
 F 1 "SW_DIP_x02" H 2350 4800 50  0000 C CNN
-F 2 "" H 2350 4950 50  0001 C CNN
+F 2 "Buttons_Switches_THT:SW_PUSH-12mm" H 2350 4950 50  0001 C CNN
 F 3 "" H 2350 4950 50  0001 C CNN
 	1    2350 4950
@@
 F 0 "R9" V 2780 4600 50  0000 C CNN
 F 1 "R" V 2700 4600 50  0000 C CNN
-F 2 "Resistors_SMD:R_0201" V 2630 4600 50  0001 C CNN
+F 2 "Resistors_THT:R_Axial_DIN0204_L3.6mm_D1.6mm_P7.62mm_Horizontal" V 2630 4600 50  0001 C CNN
 F 3 "" H 2700 4600 50  0001 C CNN
 	1    2700 4600
@@
 F 0 "SW2" H 6300 7550 50  0000 C CNN
 F 1 "SW_DIP_x02" H 6300 7150 50  0000 C CNN
-F 2 "" H 6300 7300 50  0001 C CNN
+F 2 "Buttons_Switches_THT:SW_PUSH-12mm" H 6300 7300 50  0001 C CNN
 F 3 "" H 6300 7300 50  0001 C CNN
 	1    6300 7300
@@
 F 0 "R10" V 6730 6950 50  0000 C CNN
 F 1 "R" V 6650 6950 50  0000 C CNN
-F 2 "Resistors_SMD:R_0201" V 6580 6950 50  0001 C CNN
+F 2 "Resistors_THT:R_Axial_DIN0204_L3.6mm_D1.6mm_P7.62mm_Horizontal" V 6580 6950 50  0001 C CNN
 F 3 "" H 6650 6950 50  0001 C CNN
 	1    6650 6950
@@
 F 0 "R11" V 4580 2425 50  0000 C CNN
 F 1 "R" V 4500 2425 50  0000 C CNN
-F 2 "Resistors_SMD:R_0201" V 4430 2425 50  0001 C CNN
+F 2 "Resistors_THT:R_Axial_DIN0204_L3.6mm_D1.6mm_P7.62mm_Horizontal" V 4430 2425 50  0001 C CNN
 F 3 "" H 4500 2425 50  0001 C CNN
 	1    4500 2425
