File: Agoita-aTope/PCB/PCB Display/PCBdisplay.sch (KiCad schematic (older format))
At the start: 27 parts, among them J1 CONN_02X20, SW1 SW_DIP_x02, SW2 SW_DIP_x02

Commit message: commit
Parts:
- J1: footprint Pin_Headers:Pin_Header_Angled_2x20_Pitch2.00mm -> Pin_Headers:Pin_Header_Angled_2x20_Pitch2.54mm
Connections:
- net +5V is gone; now on net +3V3: SW1.4, SW2.4
- net GND: now also DS1.16 (LED-)
- net GPIO14: now also R10.2, SW1.2; no longer D9.2 (A)
- net GPIO15: now also D9.2 (A); no longer R10.2, SW1.2
- net +3V3: now reaches J1.1 (P1)
- no-connect marks 28 -> 26
Changed lines of the file:
@@
 	1    0    0    -1
 $EndComp
-NoConn ~ 3850 7400
 NoConn ~ 4450 7400
 NoConn ~ 4550 7400
@@
 F 0 "J1" H 4400 6450 50  0000 C CNN
 F 1 "CONN_02X20" V 4400 5400 50  0000 C CNN
-F 2 "Pin_Headers:Pin_Header_Angled_2x20_Pitch2.00mm" H 4400 4450 50  0001 C CNN
+F 2 "Pin_Headers:Pin_Header_Angled_2x20_Pitch2.54mm" H 4400 4450 50  0001 C CNN
 F 3 "" H 4400 4450 50  0001 C CNN
 	1    4400 5400
@@
 GPIO20
 NoConn ~ 3550 5150
-NoConn ~ 3450 5650
 NoConn ~ 3650 5150
 NoConn ~ 4050 5150
@@
 $EndComp
 Text Label 2350 4505 1    60   ~ 0
-GPIO15
+GPIO14
 $Comp
 L Buzzer BZ1
@@
 GPIO18
 Text Label 1300 5100 3    60   ~ 0
-GPIO14
+GPIO15
 Text Label 4150 7275 1    60   ~ 0
 GPIO4
@@
 $EndComp
 $Comp
-L +5V #PWR016
+L +3.3V #PWR016
 U 1 1 595CF744
 P 6400 7650
 F 0 "#PWR016" H 6400 7500 50  0001 C CNN
-F 1 "+5V" H 6400 7790 50  0000 C CNN
+F 1 "+3.3V" H 6400 7790 50  0000 C CNN
 F 2 "" H 6400 7650 50  0001 C CNN
 F 3 "" H 6400 7650 50  0001 C CNN
@@
 $EndComp
 $Comp
-L +5V #PWR017
+L +3.3V #PWR017
 U 1 1 595CFA9D
 P 2450 5300
 F 0 "#PWR017" H 2450 5150 50  0001 C CNN
-F 1 "+5V" H 2450 5440 50  0000 C CNN
+F 1 "+3.3V" H 2450 5440 50  0000 C CNN
 F 2 "" H 2450 5300 50  0001 C CNN
 F 3 "" H 2450 5300 50  0001 C CNN
@@
 NoConn ~ 2350 5250
 NoConn ~ 2450 4650
+Wire Wire Line
+	3850 7400 3850 7280
+$Comp
+L GND #PWR018
+U 1 1 595E80E2
+P 3850 7280
+F 0 "#PWR018" H 3850 7030 50  0001 C CNN
+F 1 "GND" H 3850 7130 50  0000 C CNN
+F 2 "" H 3850 7280 50  0001 C CNN
+F 3 "" H 3850 7280 50  0001 C CNN
+	1    3850 7280
+	0    1    1    0
+$EndComp
+$Comp
+L +3.3V #PWR?
+U 1 1 595F76EE
+P 3450 5650
+F 0 "#PWR?" H 3450 5500 50  0001 C CNN
+F 1 "+3.3V" H 3450 5790 50  0000 C CNN
+F 2 "" H 3450 5650 50  0001 C CNN
+F 3 "" H 3450 5650 50  0001 C CNN
+	1    3450 5650
+	-1   0    0    1
+$EndComp
 $EndSCHEMATC

Commit message: commit
Connections:
- net GND: now also J1.39 (P39); no longer J1.25 (P25)
- net GPIO19: no longer names the net of J1.35 (P35)
- net GPIO19: no longer RV1.1
- new net +5V: RV1.1
- no-connect marks 26 -> 27
Changed lines of the file:
@@
 Text Label 4550 6000 3    60   ~ 0
 GPIO11
-Text Label 5150 6000 3    60   ~ 0
-GPIO19
 Text Label 5250 6000 3    60   ~ 0
 GPIO26
@@
 NoConn ~ 3850 5650
 NoConn ~ 4250 5650
-NoConn ~ 5350 5650
 $Comp
 L SW_DIP_x02 SW1
@@
 F 3 "" H 2805 4510 50  0001 C CNN
 	1    2805 4510
-	1    0    0    -1
-$EndComp
-$Comp
-L GND #PWR05
-U 1 1 595670DC
-P 4650 5650
-F 0 "#PWR05" H 4650 5400 50  0001 C CNN
-F 1 "GND" H 4650 5500 50  0000 C CNN
-F 2 "" H 4650 5650 50  0001 C CNN
-F 3 "" H 4650 5650 50  0001 C CNN
-	1    4650 5650
 	1    0    0    -1
 $EndComp
@@
 Text Label 6050 3180 3    60   ~ 0
 GPIO20
-Text Label 6125 4925 1    60   ~ 0
-GPIO19
 Text Label 6500 5150 0    60   ~ 0
 CONT_DISP
@@
 	4550 5650 4550 6000
 Wire Wire Line
-	5150 5650 5150 6000
-Wire Wire Line
 	5250 5650 5250 6000
 Wire Notes Line
@@
 	-1   0    0    1
 $EndComp
+NoConn ~ 5145 5650
+$Comp
+L GND #PWR?
+U 1 1 595F9C8B
+P 5350 5650
+F 0 "#PWR?" H 5350 5400 50  0001 C CNN
+F 1 "GND" H 5350 5500 50  0000 C CNN
+F 2 "" H 5350 5650 50  0001 C CNN
+F 3 "" H 5350 5650 50  0001 C CNN
+	1    5350 5650
+	1    0    0    -1
+$EndComp
+NoConn ~ 4650 5645
+$Comp
+L +5V #PWR?
+U 1 1 595FA0A6
+P 6125 4925
+F 0 "#PWR?" H 6125 4775 50  0001 C CNN
+F 1 "+5V" H 6125 5065 50  0000 C CNN
+F 2 "" H 6125 4925 50  0001 C CNN
+F 3 "" H 6125 4925 50  0001 C CNN
+	1    6125 4925
+	1    0    0    -1
+$EndComp
+$Comp
+L +5V #PWR?
+U 1 1 595FA42D
+P 7365 4705
+F 0 "#PWR?" H 7365 4555 50  0001 C CNN
+F 1 "+5V" H 7365 4845 50  0000 C CNN
+F 2 "" H 7365 4705 50  0001 C CNN
+F 3 "" H 7365 4705 50  0001 C CNN
+	1    7365 4705
+	1    0    0    -1
+$EndComp
+$Comp
+L +5V #PWR?
+U 1 1 595FA45C
+P 7365 4705
+F 0 "#PWR?" H 7365 4555 50  0001 C CNN
+F 1 "+5V" H 7365 4845 50  0000 C CNN
+F 2 "" H 7365 4705 50  0001 C CNN
+F 3 "" H 7365 4705 50  0001 C CNN
+	1    7365 4705
+	1    0    0    -1
+$EndComp
+$Comp
+L +5V #PWR?
+U 1 1 595FA470
+P 7365 4705
+F 0 "#PWR?" H 7365 4555 50  0001 C CNN
+F 1 "+5V" H 7365 4845 50  0000 C CNN
+F 2 "" H 7365 4705 50  0001 C CNN
+F 3 "" H 7365 4705 50  0001 C CNN
+	1    7365 4705
+	1    0    0    -1
+$EndComp
+$Comp
+L +5V #PWR?
+U 1 1 595FA49F
+P 7365 4705
+F 0 "#PWR?" H 7365 4555 50  0001 C CNN
+F 1 "+5V" H 7365 4845 50  0000 C CNN
+F 2 "" H 7365 4705 50  0001 C CNN
+F 3 "" H 7365 4705 50  0001 C CNN
+	1    7365 4705
+	1    0    0    -1
+$EndComp
+$Comp
+L +5V #PWR?
+U 1 1 595FA4B3
+P 7365 4705
+F 0 "#PWR?" H 7365 4555 50  0001 C CNN
+F 1 "+5V" H 7365 4845 50  0000 C CNN
+F 2 "" H 7365 4705 50  0001 C CNN
+F 3 "" H 7365 4705 50  0001 C CNN
+	1    7365 4705
+	1    0    0    -1
+$EndComp
+$Comp
+L +5V #PWR?
+U 1 1 595FA4C7
+P 7365 4705
+F 0 "#PWR?" H 7365 4555 50  0001 C CNN
+F 1 "+5V" H 7365 4845 50  0000 C CNN
+F 2 "" H 7365 4705 50  0001 C CNN
+F 3 "" H 7365 4705 50  0001 C CNN
+	1    7365 4705
+	1    0    0    -1
+$EndComp
+$Comp
+L +5V #PWR?
+U 1 1 595FA4DB
+P 7365 4705
+F 0 "#PWR?" H 7365 4555 50  0001 C CNN
+F 1 "+5V" H 7365 4845 50  0000 C CNN
+F 2 "" H 7365 4705 50  0001 C CNN
+F 3 "" H 7365 4705 50  0001 C CNN
+	1    7365 4705
+	1    0    0    -1
+$EndComp
+$Comp
+L +5V #PWR?
+U 1 1 595FA4EF
+P 7365 4705
+F 0 "#PWR?" H 7365 4555 50  0001 C CNN
+F 1 "+5V" H 7365 4845 50  0000 C CNN
+F 2 "" H 7365 4705 50  0001 C CNN
+F 3 "" H 7365 4705 50  0001 C CNN
+	1    7365 4705
+	1    0    0    -1
+$EndComp
+$Comp
+L +5V #PWR?
+U 1 1 595FA503
+P 7365 4705
+F 0 "#PWR?" H 7365 4555 50  0001 C CNN
+F 1 "+5V" H 7365 4845 50  0000 C CNN
+F 2 "" H 7365 4705 50  0001 C CNN
+F 3 "" H 7365 4705 50  0001 C CNN
+	1    7365 4705
+	1    0    0    -1
+$EndComp
+$Comp
+L +5V #PWR?
+U 1 1 595FA517
+P 7365 4705
+F 0 "#PWR?" H 7365 4555 50  0001 C CNN
+F 1 "+5V" H 7365 4845 50  0000 C CNN
+F 2 "" H 7365 4705 50  0001 C CNN
+F 3 "" H 7365 4705 50  0001 C CNN
+	1    7365 4705
+	1    0    0    -1
+$EndComp
+$Comp
+L +5V #PWR?
+U 1 1 595FA52B
+P 7365 4705
+F 0 "#PWR?" H 7365 4555 50  0001 C CNN
+F 1 "+5V" H 7365 4845 50  0000 C CNN
+F 2 "" H 7365 4705 50  0001 C CNN
+F 3 "" H 7365 4705 50  0001 C CNN
+	1    7365 4705
+	1    0    0    -1
+$EndComp
+$Comp
+L +5V #PWR?
+U 1 1 595FA53F
+P 7365 4705
+F 0 "#PWR?" H 7365 4555 50  0001 C CNN
+F 1 "+5V" H 7365 4845 50  0000 C CNN
+F 2 "" H 7365 4705 50  0001 C CNN
+F 3 "" H 7365 4705 50  0001 C CNN
+	1    7365 4705
+	1    0    0    -1
+$EndComp
+$Comp
+L +5V #PWR?
+U 1 1 595FA553
+P 7365 4705
+F 0 "#PWR?" H 7365 4555 50  0001 C CNN
+F 1 "+5V" H 7365 4845 50  0000 C CNN
+F 2 "" H 7365 4705 50  0001 C CNN
+F 3 "" H 7365 4705 50  0001 C CNN
+	1    7365 4705
+	1    0    0    -1
+$EndComp
+$Comp
+L +5V #PWR?
+U 1 1 595FA567
+P 7365 4705
+F 0 "#PWR?" H 7365 4555 50  0001 C CNN
+F 1 "+5V" H 7365 4845 50  0000 C CNN
+F 2 "" H 7365 4705 50  0001 C CNN
+F 3 "" H 7365 4705 50  0001 C CNN
+	1    7365 4705
+	1    0    0    -1
+$EndComp
+$Comp
+L +5V #PWR?
+U 1 1 595FA57B
+P 7365 4705
+F 0 "#PWR?" H 7365 4555 50  0001 C CNN
+F 1 "+5V" H 7365 4845 50  0000 C CNN
+F 2 "" H 7365 4705 50  0001 C CNN
+F 3 "" H 7365 4705 50  0001 C CNN
+	1    7365 4705
+	1    0    0    -1
+$EndComp
 $EndSCHEMATC
